Commit message: Add hardware interface for stmbot robot

File: robot-ros2-packages/stmbot_description/urdf/stmbot.urdf.xacro (robot description, xacro)
@@ -1,4 +1,5 @@
 <?xml version="1.0"?>
 <robot xmlns:xacro="http://www.ros.org/wiki/xacro" name="stmbot">
+    <xacro:arg name="is_sim" default="true"/>
     <xacro:include filename="$(find stmbot_description)/urdf/stmbot_gazebo.xacro" />
     <!-- Include ros2_control Plugins -->

File: robot-ros2-packages/stmbot_description/urdf/stmbot_ros2_control.xacro (robot description, xacro)
@@ -3,7 +3,23 @@
     <ros2_control name="RobotSystem" type="system">
         <xacro:property name="PI" value="3.14159265359" />
-        <hardware>
-            <plugin>gazebo_ros2_control/GazeboSystem</plugin>
-        </hardware>
+        <xacro:if value="$(arg is_sim)">
+            <hardware>
+                <plugin>gazebo_ros2_control/GazeboSystem</plugin>
+                <joint name="joint_5">
+                    <param name="mimic">joint_4</param>
+                    <param name="multiplier">-1</param>
+                    <command_interface name="position">
+                        <param name="min">0.0</param>
+                        <param name="max">${PI / 2}</param>
+                    </command_interface>
+                </joint>
+            </hardware>
+        </xacro:if>
+        <xacro:unless value="$(arg is_sim)">
+            <hardware>
+                <plugin>stmbot_controllers/StmbotInterface</plugin>
+                <param name="port">/dev/ttyUSB0</param>
+            </hardware>
+        </xacro:unless>
         <joint name="joint_1">
             <command_interface name="position">
@@ -34,12 +50,4 @@
             <state_interface name="position" />
         </joint>
-        <joint name="joint_5">
-            <param name="mimic">joint_4</param>
-            <param name="multiplier">-1</param>
-            <command_interface name="position">
-                <param name="min">0.0</param>
-                <param name="max">${PI / 2}</param>
-            </command_interface>
-        </joint>
     </ros2_control>
 </robot>
